Commit message: basic ros-control integration

File: jet_description/urdf/jet.xacro (robot description, xacro)
@@ -90,23 +90,25 @@
     </inertial>
   </link>
-  <joint name="base_to_right_wheel" type="continuous">
+  <joint name="right_wheel_joint" type="revolute">
     <parent link="base_link"/>
     <child link="right_wheel"/>
     <origin xyz="0.15 -.05 -.03"/>
     <axis xyz="1 0 0"/>
+    <limit effort="100" velocity="100.0" lower="-5000" upper="5000" />
   </joint>
-  <joint name="base_to_left_wheel" type="continuous">
+  <joint name="left_wheel_joint" type="revolute">
     <parent link="base_link"/>
     <child link="left_wheel"/>
     <origin xyz="-0.15 -.05 -.03"/>
     <axis xyz="1 0 0"/>
+    <limit effort="100" velocity="100.0" lower="-5000" upper="5000"/>
   </joint>
   <transmission name="tran_left_wheel">
     <type>transmission_interface/SimpleTransmission</type>
-    <joint name="base_to_right_wheel">
-      <hardwareInterface>EffortJointInterface</hardwareInterface>
+    <joint name="left_wheel_joint">
+      <hardwareInterface>VelocityJointInterface</hardwareInterface>
     </joint>
-    <actuator name="motor_right">
-      <hardwareInterface>EffortJointInterface</hardwareInterface>
+    <actuator name="motor_left">
+      <hardwareInterface>VelocityJointInterface</hardwareInterface>
       <mechanicalReduction>1</mechanicalReduction>
     </actuator>
@@ -114,9 +116,9 @@
   <transmission name="tran_right_wheel">
     <type>transmission_interface/SimpleTransmission</type>
-    <joint name="base_to_left_wheel">
-      <hardwareInterface>EffortJointInterface</hardwareInterface>
+    <joint name="right_wheel_joint">
+      <hardwareInterface>VelocityJointInterface</hardwareInterface>
     </joint>
-    <actuator name="motor_left">
-      <hardwareInterface>EffortJointInterface</hardwareInterface>
+    <actuator name="motor_right">
+      <hardwareInterface>VelocityJointInterface</hardwareInterface>
       <mechanicalReduction>1</mechanicalReduction>
     </actuator>

Commit message: fixed diff drive in gazebo

File: jet_description/urdf/jet.xacro (robot description, xacro)
@@ -22,7 +22,15 @@
     </collision>
     <inertial>
-      <mass value="10"/>
-      <inertia ixx="5e-3" ixy="0.0" ixz="0.0" iyy="5e-3" iyz="0.0" izz="5e-3"/>
+      <mass value="1"/>
+      <inertia ixx="1e-3" ixy="0.0" ixz="0.0" iyy="1e-3" iyz="0.0" izz="1e-3"/>
     </inertial>
+  </link>
+  <link name="caster">
+    <visual name='caster_visual'>
+      <origin rpy="0 0 0" xyz="0 .15 -.06"/>
+      <geometry>
+        <cylinder radius="0.03" length="0.12"/>
+      </geometry>
+    </visual>
     <collision name='caster_collision'>
       <origin rpy="0 0 0" xyz="0 .15 -.06"/>
@@ -41,10 +49,8 @@
       </surface>
     </collision>
-    <visual name='caster_visual'>
-      <origin rpy="0 0 0" xyz="0 .15 -.06"/>
-      <geometry>
-        <cylinder radius="0.03" length="0.12"/>
-      </geometry>
-    </visual>
+    <inertial>
+      <mass value="10"/>
+      <inertia ixx=".01425" ixy="0.0" ixz="0.0" iyy=".01425" iyz="0.0" izz=".0045"/>
+    </inertial>
   </link>
   <link name="right_wheel">
@@ -65,5 +71,5 @@
     </collision>
     <inertial>
-      <mass value="10"/>
+      <mass value="1"/>
       <inertia ixx="1e-3" ixy="0.0" ixz="0.0" iyy="1e-3" iyz="0.0" izz="1e-3"/>
     </inertial>
@@ -90,4 +96,10 @@
     </inertial>
   </link>
+  <joint name="caster_base_joint" type="fixed">
+    <parent link="base_link"/>
+    <child link="caster"/>
+    <origin xyz="0 0 0"/>
+    <axis xyz="0 0 1"/>
+  </joint>
   <joint name="right_wheel_joint" type="revolute">
     <parent link="base_link"/>

Commit message: added camera sensor to gazebo

File: jet_description/urdf/jet.xacro (robot description, xacro)
@@ -96,4 +96,32 @@
     </inertial>
   </link>
+  <link name="camera_link">
+    <collision>
+      <origin xyz="0 0 0" rpy="0 0 0"/>
+      <geometry>
+        <box size=".05 .02 .05"/>
+      </geometry>
+    </collision>
+    <visual>
+      <origin xyz="0 0 0" rpy="0 0 0"/>
+      <geometry>
+        <box size=".05 .02 .05"/>
+      </geometry>
+      <material name="red">
+        <color rgba="1.0 0 0 1"/>
+      </material>
+    </visual>
+    <inertial>
+      <mass value="1e-5" />
+      <origin xyz="0 0 0" rpy="0 0 0"/>
+      <inertia ixx="1e-6" ixy="0" ixz="0" iyy="1e-6" iyz="0" izz="1e-6" />
+    </inertial>
+  </link>
+  <joint name="camera_joint" type="fixed">
+      <axis xyz="0 1 0" />
+      <origin xyz="0 -.15 .05" rpy="0 0 0"/>
+      <parent link="base_link"/>
+      <child link="camera_link"/>
+  </joint>
   <joint name="caster_base_joint" type="fixed">
     <parent link="base_link"/>

Commit message: sonar sensors in gazebo

File: jet_description/urdf/jet.xacro (robot description, xacro)
@@ -96,7 +96,28 @@
     </inertial>
   </link>
+  <link name="sonar1_link">
+    <inertial>
+      <mass value="1e-5" />
+      <origin xyz="0 0 0" rpy="0 0 0"/>
+      <inertia ixx="1e-6" ixy="0" ixz="0" iyy="1e-6" iyz="0" izz="1e-6" />
+    </inertial>
+  </link>
+  <link name="sonar2_link">
+    <inertial>
+      <mass value="1e-5" />
+      <origin xyz="0 0 0" rpy="0 0 0"/>
+      <inertia ixx="1e-6" ixy="0" ixz="0" iyy="1e-6" iyz="0" izz="1e-6" />
+    </inertial>
+  </link>
+  <link name="sonar3_link">
+    <inertial>
+      <mass value="1e-5" />
+      <origin xyz="0 0 0" rpy="0 0 0"/>
+      <inertia ixx="1e-6" ixy="0" ixz="0" iyy="1e-6" iyz="0" izz="1e-6" />
+    </inertial>
+  </link>
   <link name="camera_link">
     <collision>
-      <origin xyz="0 0 0" rpy="0 0 0"/>
+      <origin xyz="0 0 0" rpy="0 0 -1.57075"/>
       <geometry>
         <box size=".05 .02 .05"/>
@@ -104,5 +125,5 @@
     </collision>
     <visual>
-      <origin xyz="0 0 0" rpy="0 0 0"/>
+      <origin xyz="0 0 0" rpy="0 0 -1.57075"/>
       <geometry>
         <box size=".05 .02 .05"/>
@@ -118,4 +139,22 @@
     </inertial>
   </link>
+  <joint name="sonar1_joint" type="fixed">
+      <axis xyz="0 1 0" />
+      <origin xyz="-.1 -.15 -.05" rpy="0 0 -2.356125"/>
+      <parent link="base_link"/>
+      <child link="sonar1_link"/>
+  </joint>
+  <joint name="sonar2_joint" type="fixed">
+      <axis xyz="0 1 0" />
+      <origin xyz="0 -.15 -.05" rpy="0 0 -1.57075"/>
+      <parent link="base_link"/>
+      <child link="sonar2_link"/>
+  </joint>
+  <joint name="sonar3_joint" type="fixed">
+      <axis xyz="0 1 0" />
+      <origin xyz=".1 -.15 -.05" rpy="0 0 -.785375"/>
+      <parent link="base_link"/>
+      <child link="sonar3_link"/>
+  </joint>
   <joint name="camera_joint" type="fixed">
       <axis xyz="0 1 0" />

Commit message: gazebo imu sensor

File: jet_description/urdf/jet.xacro (robot description, xacro)
@@ -139,4 +139,17 @@
     </inertial>
   </link>
+  <link name="gyro_link">
+    <inertial>
+      <mass value="0.001"/>
+      <origin rpy="0 0 0" xyz="0 0 0"/>
+      <inertia ixx="0.0001" ixy="0" ixz="0" iyy="0.000001" iyz="0" izz="0.0001"/>
+    </inertial>
+  </link>
+  <joint name="imu_joint" type="fixed">
+    <axis xyz="1 0 0"/>
+    <origin xyz="0 0 0"/>
+    <parent link="base_link"/>
+    <child link="gyro_link"/>
+  </joint>
   <joint name="sonar1_joint" type="fixed">
       <axis xyz="0 1 0" />
